File: hardware/analog/analog.sch (KiCad schematic (older format))
At the start: 5 parts, among them J1 RTD conn, J2 DAQ CONN, J3 RTD conn, J4 Laser Diode Conn, J5 Barrel_Jack

Commit message: Refine analog circuitry
Parts:
- removed J2: DAQ CONN, symbol Connector:Conn_01x05_Female
- added J?: Conn_01x06_Female, symbol Connector:Conn_01x06_Female
Connections:
- wire segments 22 -> 25
Other:
- note added: "High Level Connections"
- note added: "outputs between +/- 0.75V"
Changed lines of the file:
@@
 $Descr A4 11693 8268
 encoding utf-8
-Sheet 1 6
+Sheet 1 7
 Title ""
 Date ""
@@
 F2 "LD_POWER" I L 7950 5350 50
 F3 "PD_SIGNAL" I L 7950 5250 50
-F4 "SMI_SIGNAL" I L 7950 4700 50
+F4 "SMI_SIGNAL_AC" I L 7950 4850 50
+F5 "SMI_SIGNAL_DC" I L 7950 4700 50
 $EndSheet
 $Comp
@@
 Text Notes 6300 5400 0    50   ~ 0
 to laser diode\n(offboard)
-$Comp
-L Connector:Conn_01x05_Female J2
-U 1 1 5D905FF1
-P 8300 1800
-F 0 "J2" H 8327 1826 50  0000 L CNN
-F 1 "DAQ CONN" H 8327 1735 50  0000 L CNN
-F 2 "" H 8300 1800 50  0001 C CNN
-F 3 "~" H 8300 1800 50  0001 C CNN
-	1    8300 1800
-	1    0    0    -1
-$EndComp
 Wire Wire Line
 	7200 5250 7950 5250
@@
 	5600 4700 5600 1800
 Wire Wire Line
-	7950 4700 5750 4700
-Wire Wire Line
-	5750 4700 5750 1900
-Wire Wire Line
 	5750 1900 8100 1900
 $Comp
 L power:GNDREF #PWR01
 U 1 1 5D907722
-P 7150 2300
-F 0 "#PWR01" H 7150 2050 50  0001 C CNN
-F 1 "GNDREF" H 7155 2127 50  0000 C CNN
-F 2 "" H 7150 2300 50  0001 C CNN
-F 3 "" H 7150 2300 50  0001 C CNN
-	1    7150 2300
+P 7150 2400
+F 0 "#PWR01" H 7150 2150 50  0001 C CNN
+F 1 "GNDREF" H 7155 2227 50  0000 C CNN
+F 2 "" H 7150 2400 50  0001 C CNN
+F 3 "" H 7150 2400 50  0001 C CNN
+	1    7150 2400
 	1    0    0    -1
 $EndComp
 Wire Wire Line
-	7150 2300 7150 2000
+	7150 2400 7150 2100
 Wire Wire Line
-	7150 2000 8100 2000
+	7150 2100 8100 2100
+Wire Wire Line
+	7950 4850 5750 4850
+Wire Wire Line
+	5750 1900 5750 4850
+$Comp
+L Connector:Conn_01x06_Female J?
+U 1 1 5DAC4DEB
+P 8300 1800
+F 0 "J?" H 8327 1776 50  0000 L CNN
+F 1 "Conn_01x06_Female" H 8327 1685 50  0000 L CNN
+F 2 "" H 8300 1800 50  0001 C CNN
+F 3 "~" H 8300 1800 50  0001 C CNN
+	1    8300 1800
+	1    0    0    -1
+$EndComp
+Wire Wire Line
+	7950 4700 5900 4700
+Wire Wire Line
+	5900 4700 5900 2000
+Wire Wire Line
+	5900 2000 8100 2000
+Text Notes 6500 1500 0    50   ~ 0
+outputs between +/- 0.75V
+Text Notes 5100 900  0    100  ~ 20
+High Level Connections
 $EndSCHEMATC

Commit message: Save filters and whatnot before the culling
TODO:
- split ambient and SMI circuitry onto different boards
- kill off the pseudoground and use lipo batteries instead
Parts:
- J1, J3: footprint (none) -> Connectors_Phoenix:PhoenixContact_MCV-G_02x3.50mm_Vertical
- J2: renamed from J?; footprint (none) -> Connectors_Phoenix:PhoenixContact_MCV-G_06x3.50mm_Vertical
- J4: footprint (none) -> Connectors_Phoenix:PhoenixContact_MCV-G_03x3.50mm_Vertical
- J5: footprint (none) -> Connect:BARREL_JACK
Changed lines of the file:
@@
 F 0 "J5" H 1555 6825 50  0000 C CNN
 F 1 "Barrel_Jack" H 1555 6734 50  0000 C CNN
-F 2 "" H 1550 6460 50  0001 C CNN
+F 2 "Connect:BARREL_JACK" H 1550 6460 50  0001 C CNN
 F 3 "~" H 1550 6460 50  0001 C CNN
 	1    1500 6500
@@
 F 0 "J1" H 1644 1325 50  0000 C CNN
 F 1 "RTD conn" H 1644 1416 50  0000 C CNN
-F 2 "" H 1750 1650 50  0001 C CNN
+F 2 "Connectors_Phoenix:PhoenixContact_MCV-G_02x3.50mm_Vertical" H 1750 1650 50  0001 C CNN
 F 3 "~" H 1750 1650 50  0001 C CNN
 	1    1750 1650
@@
 F 0 "J3" H 1644 2525 50  0000 C CNN
 F 1 "RTD conn" H 1644 2616 50  0000 C CNN
-F 2 "" H 1750 2850 50  0001 C CNN
+F 2 "Connectors_Phoenix:PhoenixContact_MCV-G_02x3.50mm_Vertical" H 1750 2850 50  0001 C CNN
 F 3 "~" H 1750 2850 50  0001 C CNN
 	1    1750 2850
@@
 F 0 "J4" H 6894 5025 50  0000 C CNN
 F 1 "Laser Diode Conn" H 6894 5116 50  0000 C CNN
-F 2 "" H 7000 5350 50  0001 C CNN
+F 2 "Connectors_Phoenix:PhoenixContact_MCV-G_03x3.50mm_Vertical" H 7000 5350 50  0001 C CNN
 F 3 "~" H 7000 5350 50  0001 C CNN
 	1    7000 5350
@@
 	5750 1900 5750 4850
 $Comp
-L Connector:Conn_01x06_Female J?
+L Connector:Conn_01x06_Female J2
 U 1 1 5DAC4DEB
 P 8300 1800
-F 0 "J?" H 8327 1776 50  0000 L CNN
+F 0 "J2" H 8327 1776 50  0000 L CNN
 F 1 "Conn_01x06_Female" H 8327 1685 50  0000 L CNN
-F 2 "" H 8300 1800 50  0001 C CNN
+F 2 "Connectors_Phoenix:PhoenixContact_MCV-G_06x3.50mm_Vertical" H 8300 1800 50  0001 C CNN
 F 3 "~" H 8300 1800 50  0001 C CNN
 	1    8300 1800
