File: hardware/analog/power.sch (KiCad schematic (older format))
At the start: 17 parts, among them Q1 Q_NPN_EBC, U01 +18V, U2 BUF634A, U3 TL081

Commit message: Refine analog circuitry
Parts:
- added U13: L7818, symbol Regulator_Linear:L7818
Connections:
- wire segments 60 -> 63
Other:
- note added: "(capacitor multiplier: not \nimplemented, may remove)"
- note added: "+18V & +9V intentionally shorted"
- note added: "GNDPWR & -9V intentionally shorted"
- note removed: "Alternative: put pos/neg regulator\npair here."
- note removed: "Regulation stage, maybe"
- moved on the sheet: U3

Commit message: Save filters and whatnot before the culling
TODO:
- split ambient and SMI circuitry onto different boards
- kill off the pseudoground and use lipo batteries instead
Parts:
- removed U01: +18V, symbol smi:+18V
- C1, C2, C5, C6, C7: footprint (none) -> Capacitor_SMD:C_0805_2012Metric_Pad1.15x1.40mm_HandSolder
- C3, C4: footprint (none) -> Capacitor_THT:CP_Radial_D8.0mm_P3.80mm
- FB1: footprint (none) -> Resistor_THT:R_Axial_DIN0204_L3.6mm_D1.6mm_P7.62mm_Horizontal
- Q1: footprint (none) -> Package_TO_SOT_SMD:SOT-23_Handsoldering
- R1, R2, R3, R4: footprint (none) -> Resistor_SMD:R_0805_2012Metric_Pad1.15x1.40mm_HandSolder
- U13: footprint (none) -> TO_SOT_Packages_THT:TO-220-3_Vertical
- U2, U3: footprint (none) -> Housings_SOIC:SOIC-8_3.9x4.9mm_Pitch1.27mm
Connections:
- net labels added: +18V
Changed lines of the file:
@@
 PWR-
-$Comp
-L Device:Q_NPN_EBC Q?
-U 1 1 5D8E7401
-P 2600 2650
-AR Path="/5D8E7401" Ref="Q?"  Part="1"
-AR Path="/5D8E6431/5D8E7401" Ref="Q1"  Part="1"
-F 0 "Q1" V 2928 2650 50  0000 C CNN
-F 1 "Q_NPN_EBC" V 2837 2650 50  0000 C CNN
-F 2 "" H 2800 2750 50  0001 C CNN
-F 3 "~" H 2600 2650 50  0001 C CNN
-	1    2600 2650
-	0    -1   -1   0
-$EndComp
-$Comp
-L Device:Ferrite_Bead_Small FB?
-U 1 1 5D8E7409
-P 2600 2950
-AR Path="/5D8E7409" Ref="FB?"  Part="1"
-AR Path="/5D8E6431/5D8E7409" Ref="FB1"  Part="1"
-F 0 "FB1" H 2700 2950 50  0000 L CNN
-F 1 "F" H 2700 2905 50  0001 L CNN
-F 2 "" V 2530 2950 50  0001 C CNN
-F 3 "~" H 2600 2950 50  0001 C CNN
-	1    2600 2950
-	1    0    0    -1
-$EndComp
-$Comp
-L Device:R_US R?
-U 1 1 5D8E7410
-P 2150 2850
-AR Path="/5D8E7410" Ref="R?"  Part="1"
-AR Path="/5D8E6431/5D8E7410" Ref="R1"  Part="1"
-F 0 "R1" H 2218 2896 50  0000 L CNN
-F 1 "R_US" H 2218 2805 50  0000 L CNN
-F 2 "" V 2190 2840 50  0001 C CNN
-F 3 "~" H 2150 2850 50  0001 C CNN
-	1    2150 2850
-	1    0    0    -1
-$EndComp
-$Comp
-L Device:C C?
-U 1 1 5D8E7417
-P 2150 3800
-AR Path="/5D8E7417" Ref="C?"  Part="1"
-AR Path="/5D8E6431/5D8E7417" Ref="C4"  Part="1"
-F 0 "C4" H 2265 3846 50  0000 L CNN
-F 1 "C" H 2265 3755 50  0000 L CNN
-F 2 "" H 2188 3650 50  0001 C CNN
-F 3 "~" H 2150 3800 50  0001 C CNN
-	1    2150 3800
-	1    0    0    -1
-$EndComp
-Wire Wire Line
-	2150 2700 2150 2550
-Connection ~ 2150 2550
-Wire Wire Line
-	2150 2550 2400 2550
-$Comp
-L Diode:1N4001 D?
-U 1 1 5D8E7421
-P 3000 3700
-AR Path="/5D8E7421" Ref="D?"  Part="1"
-AR Path="/5D8E6431/5D8E7421" Ref="D1"  Part="1"
-F 0 "D1" V 3046 3621 50  0000 R CNN
-F 1 "1N4001" V 2955 3621 50  0000 R CNN
-F 2 "Diode_THT:D_DO-41_SOD81_P10.16mm_Horizontal" H 3000 3525 50  0001 C CNN
-F 3 "http://www.vishay.com/docs/88503/1n4001.pdf" H 3000 3700 50  0001 C CNN
-	1    3000 3700
-	0    -1   -1   0
-$EndComp
-Wire Wire Line
-	3000 3550 3000 2550
-Wire Wire Line
-	3000 2550 2800 2550
 $Comp
 L Device:C C?
@@
 F 0 "C3" H 4265 3746 50  0000 L CNN
 F 1 "220uF" H 4265 3655 50  0000 L CNN
-F 2 "" H 4188 3550 50  0001 C CNN
+F 2 "Capacitor_THT:CP_Radial_D8.0mm_P3.80mm" H 4188 3550 50  0001 C CNN
 F 3 "~" H 4150 3700 50  0001 C CNN
 	1    4150 3700
@@
 Wire Wire Line
 	4150 2550 4150 3550
-Connection ~ 3000 2550
 $Comp
 L Device:R_US R?
@@
 F 0 "R2" H 6068 3146 50  0000 L CNN
 F 1 "220K, 1%" H 6068 3055 50  0000 L CNN
-F 2 "" V 6040 3090 50  0001 C CNN
+F 2 "Resistor_SMD:R_0805_2012Metric_Pad1.15x1.40mm_HandSolder" V 6040 3090 50  0001 C CNN
 F 3 "~" H 6000 3100 50  0001 C CNN
 	1    6000 3100
@@
 F 0 "R4" H 6068 4396 50  0000 L CNN
 F 1 "220K, 1%" H 6068 4305 50  0000 L CNN
-F 2 "" V 6040 4340 50  0001 C CNN
+F 2 "Resistor_SMD:R_0805_2012Metric_Pad1.15x1.40mm_HandSolder" V 6040 4340 50  0001 C CNN
 F 3 "~" H 6000 4350 50  0001 C CNN
 	1    6000 4350
@@
 Wire Wire Line
 	4150 3850 4150 4800
-Wire Wire Line
-	3000 3850 3000 4800
-Wire Wire Line
-	1700 4800 2150 4800
-Connection ~ 3000 4800
-Wire Wire Line
-	3000 4800 3950 4800
-Wire Wire Line
-	2150 3000 2150 3350
-Wire Wire Line
-	2600 3350 2150 3350
-Wire Wire Line
-	2600 3050 2600 3350
-Connection ~ 2150 3350
-Wire Wire Line
-	2150 3350 2150 3650
-Wire Wire Line
-	2150 3950 2150 4800
-Connection ~ 2150 4800
-Wire Wire Line
-	2150 4800 3000 4800
 Wire Wire Line
 	6000 4500 6000 4800
@@
 F 0 "U3" H 7641 3796 50  0000 L CNN
 F 1 "TL081" H 7641 3705 50  0000 L CNN
-F 2 "" H 7350 3800 50  0001 C CNN
+F 2 "Housings_SOIC:SOIC-8_3.9x4.9mm_Pitch1.27mm" H 7350 3800 50  0001 C CNN
 F 3 "http://www.ti.com/lit/ds/symlink/tl081.pdf" H 7450 3900 50  0001 C CNN
 	1    7300 3750
@@
 F 0 "R3" V 7995 3750 50  0000 C CNN
 F 1 "100" V 8086 3750 50  0000 C CNN
-F 2 "" V 8240 3740 50  0001 C CNN
+F 2 "Resistor_SMD:R_0805_2012Metric_Pad1.15x1.40mm_HandSolder" V 8240 3740 50  0001 C CNN
 F 3 "~" H 8200 3750 50  0001 C CNN
 	1    8200 3750
@@
 F 0 "C5" H 8065 3996 50  0000 L CNN
 F 1 "10pF" H 8065 3905 50  0000 L CNN
-F 2 "" H 7988 3800 50  0001 C CNN
+F 2 "Capacitor_SMD:C_0805_2012Metric_Pad1.15x1.40mm_HandSolder" H 7988 3800 50  0001 C CNN
 F 3 "~" H 7950 3950 50  0001 C CNN
 	1    7950 3950
@@
 F 0 "U2" H 9541 3746 50  0000 L CNN
 F 1 "BUF634A" H 9541 3655 50  0000 L CNN
-F 2 "" H 9000 3700 50  0001 C CNN
+F 2 "Housings_SOIC:SOIC-8_3.9x4.9mm_Pitch1.27mm" H 9000 3700 50  0001 C CNN
 F 3 "" H 9000 3700 50  0001 C CNN
 	1    9000 3700
@@
 F 0 "C7" V 7171 4550 50  0000 C CNN
 F 1 "0.1uF" V 7262 4550 50  0000 C CNN
-F 2 "" H 7400 4550 50  0001 C CNN
+F 2 "Capacitor_SMD:C_0805_2012Metric_Pad1.15x1.40mm_HandSolder" H 7400 4550 50  0001 C CNN
 F 3 "~" H 7400 4550 50  0001 C CNN
 	1    7400 4550
@@
 F 0 "C1" V 7171 3100 50  0000 C CNN
 F 1 "0.1uF" V 7262 3100 50  0000 C CNN
-F 2 "" H 7400 3100 50  0001 C CNN
+F 2 "Capacitor_SMD:C_0805_2012Metric_Pad1.15x1.40mm_HandSolder" H 7400 3100 50  0001 C CNN
 F 3 "~" H 7400 3100 50  0001 C CNN
 	1    7400 3100
@@
 F 0 "C2" V 9021 3150 50  0000 C CNN
 F 1 "0.1uF" V 9112 3150 50  0000 C CNN
-F 2 "" H 9250 3150 50  0001 C CNN
+F 2 "Capacitor_SMD:C_0805_2012Metric_Pad1.15x1.40mm_HandSolder" H 9250 3150 50  0001 C CNN
 F 3 "~" H 9250 3150 50  0001 C CNN
 	1    9250 3150
@@
 F 0 "C6" V 9021 4500 50  0000 C CNN
 F 1 "0.1uF" V 9112 4500 50  0000 C CNN
-F 2 "" H 9250 4500 50  0001 C CNN
+F 2 "Capacitor_SMD:C_0805_2012Metric_Pad1.15x1.40mm_HandSolder" H 9250 4500 50  0001 C CNN
 F 3 "~" H 9250 4500 50  0001 C CNN
 	1    9250 4500
@@
 Wire Wire Line
 	9050 4500 9050 4800
-Wire Wire Line
-	1700 2550 2150 2550
 $Comp
 L power:GNDPWR #PWR010
@@
 	3950 4800 4150 4800
 $Comp
-L smi:+18V U01
+L smi:+18V #U01
 U 1 1 5D8F2BC9
 P 3950 2150
-F 0 "U01" H 3950 2150 50  0001 C CNN
+F 0 "#U01" H 3950 2150 50  0001 C CNN
 F 1 "+18V" H 4008 2137 50  0000 L CNN
 F 2 "" H 3950 2150 50  0001 C CNN
@@
 Text Notes 6600 4900 0    50   ~ 0
 GNDPWR & -9V intentionally shorted
-Wire Wire Line
-	3000 2550 3950 2550
 Connection ~ 3950 2550
 Connection ~ 3950 4800
@@
 F 0 "U13" H 5100 2792 50  0000 C CNN
 F 1 "L7818" H 5100 2701 50  0000 C CNN
-F 2 "" H 5125 2400 50  0001 L CIN
+F 2 "TO_SOT_Packages_THT:TO-220-3_Vertical" H 5125 2400 50  0001 L CIN
 F 3 "http://www.st.com/content/ccc/resource/technical/document/datasheet/41/4f/b3/b0/12/d4/47/88/CD00000444.pdf/files/CD00000444.pdf/jcr:content/translations/en.CD00000444.pdf" H 5100 2500 50  0001 C CNN
 	1    5100 2550
@@
 Text Notes 1800 5050 0    50   ~ 0
 (capacitor multiplier: not \nimplemented, may remove)
+Wire Wire Line
+	1700 2550 2150 2550
+Wire Wire Line
+	2150 2550 2400 2550
+Connection ~ 2150 2550
+Wire Wire Line
+	2150 2700 2150 2550
+Wire Wire Line
+	1700 4800 2150 4800
+Connection ~ 2150 4800
+Wire Wire Line
+	2150 3950 2150 4800
+Wire Wire Line
+	2150 3350 2150 3650
+Wire Wire Line
+	2600 3050 2600 3350
+Wire Wire Line
+	2600 3350 2150 3350
+Connection ~ 2150 3350
+Wire Wire Line
+	2150 3000 2150 3350
+Wire Wire Line
+	2150 4800 3000 4800
+Wire Wire Line
+	3000 4800 3950 4800
+Connection ~ 3000 4800
+Wire Wire Line
+	3000 3850 3000 4800
+Wire Wire Line
+	3000 2550 3950 2550
+Wire Wire Line
+	3000 2550 2800 2550
+Connection ~ 3000 2550
+Wire Wire Line
+	3000 3550 3000 2550
+$Comp
+L Diode:1N4001 D?
+U 1 1 5D8E7421
+P 3000 3700
+AR Path="/5D8E7421" Ref="D?"  Part="1"
+AR Path="/5D8E6431/5D8E7421" Ref="D1"  Part="1"
+F 0 "D1" V 3046 3621 50  0000 R CNN
+F 1 "1N4001" V 2955 3621 50  0000 R CNN
+F 2 "Diode_THT:D_DO-41_SOD81_P10.16mm_Horizontal" H 3000 3525 50  0001 C CNN
+F 3 "http://www.vishay.com/docs/88503/1n4001.pdf" H 3000 3700 50  0001 C CNN
+	1    3000 3700
+	0    -1   -1   0
+$EndComp
+$Comp
+L Device:C C?
+U 1 1 5D8E7417
+P 2150 3800
+AR Path="/5D8E7417" Ref="C?"  Part="1"
+AR Path="/5D8E6431/5D8E7417" Ref="C4"  Part="1"
+F 0 "C4" H 2265 3846 50  0000 L CNN
+F 1 "C" H 2265 3755 50  0000 L CNN
+F 2 "Capacitor_THT:CP_Radial_D8.0mm_P3.80mm" H 2188 3650 50  0001 C CNN
+F 3 "~" H 2150 3800 50  0001 C CNN
+	1    2150 3800
+	1    0    0    -1
+$EndComp
+$Comp
+L Device:R_US R?
+U 1 1 5D8E7410
+P 2150 2850
+AR Path="/5D8E7410" Ref="R?"  Part="1"
+AR Path="/5D8E6431/5D8E7410" Ref="R1"  Part="1"
+F 0 "R1" H 2218 2896 50  0000 L CNN
+F 1 "R_US" H 2218 2805 50  0000 L CNN
+F 2 "Resistor_SMD:R_0805_2012Metric_Pad1.15x1.40mm_HandSolder" V 2190 2840 50  0001 C CNN
+F 3 "~" H 2150 2850 50  0001 C CNN
+	1    2150 2850
+	1    0    0    -1
+$EndComp
+$Comp
+L Device:Ferrite_Bead_Small FB?
+U 1 1 5D8E7409
+P 2600 2950
+AR Path="/5D8E7409" Ref="FB?"  Part="1"
+AR Path="/5D8E6431/5D8E7409" Ref="FB1"  Part="1"
+F 0 "FB1" H 2700 2950 50  0000 L CNN
+F 1 "F" H 2700 2905 50  0001 L CNN
+F 2 "Resistor_THT:R_Axial_DIN0204_L3.6mm_D1.6mm_P7.62mm_Horizontal" V 2530 2950 50  0001 C CNN
+F 3 "~" H 2600 2950 50  0001 C CNN
+	1    2600 2950
+	1    0    0    -1
+$EndComp
+$Comp
+L Device:Q_NPN_EBC Q?
+U 1 1 5D8E7401
+P 2600 2650
+AR Path="/5D8E7401" Ref="Q?"  Part="1"
+AR Path="/5D8E6431/5D8E7401" Ref="Q1"  Part="1"
+F 0 "Q1" V 2928 2650 50  0000 C CNN
+F 1 "Q_NPN_EBC" V 2837 2650 50  0000 C CNN
+F 2 "Package_TO_SOT_SMD:SOT-23_Handsoldering" H 2800 2750 50  0001 C CNN
+F 3 "~" H 2600 2650 50  0001 C CNN
+	1    2600 2650
+	0    -1   -1   0
+$EndComp
 $EndSCHEMATC
