File: hardware/analog/pressure.sch (KiCad schematic (older format))
At the start: 5 parts, among them U7 MPXA6115A

Commit message: Save filters and whatnot before the culling
TODO:
- split ambient and SMI circuitry onto different boards
- kill off the pseudoground and use lipo batteries instead
Parts:
- added U1: LT1460, TO_SOT_Packages_SMD:SOT-23_Handsoldering, symbol smi:LT1460
- C9: footprint (none) -> Capacitor_SMD:C_0805_2012Metric_Pad1.15x1.40mm_HandSolder
- R10, R11, R9: footprint (none) -> Resistor_SMD:R_0805_2012Metric_Pad1.15x1.40mm_HandSolder
- U7: footprint (none) -> Housings_DIP:SMDIP-8_W9.53mm
Connections:
- net labels added: +18V
- wire segments 16 -> 20
Changed lines of the file:
@@
 F 0 "U7" H 5020 3596 50  0000 R CNN
 F 1 "MPXA6115A" H 5020 3505 50  0000 R CNN
-F 2 "" H 4950 3200 50  0001 C CNN
+F 2 "Housings_DIP:SMDIP-8_W9.53mm" H 4950 3200 50  0001 C CNN
 F 3 "http://www.nxp.com/files/sensors/doc/data_sheet/MPXA6115A.pdf" H 5450 4150 50  0001 C CNN
 	1    5450 3550
@@
 L power:+5V #PWR015
 U 1 1 5D8EF8B9
-P 5450 2950
-F 0 "#PWR015" H 5450 2800 50  0001 C CNN
-F 1 "+5V" H 5465 3123 50  0000 C CNN
-F 2 "" H 5450 2950 50  0001 C CNN
-F 3 "" H 5450 2950 50  0001 C CNN
-	1    5450 2950
+P 5450 2500
+F 0 "#PWR015" H 5450 2350 50  0001 C CNN
+F 1 "+5V" H 5465 2673 50  0000 C CNN
+F 2 "" H 5450 2500 50  0001 C CNN
+F 3 "" H 5450 2500 50  0001 C CNN
+	1    5450 2500
 	1    0    0    -1
 $EndComp
-Wire Wire Line
-	5450 2950 5450 3050
 $Comp
 L Device:C_Small C9
@@
 F 0 "C9" V 4921 3050 50  0000 C CNN
 F 1 "C_Small" V 5012 3050 50  0000 C CNN
-F 2 "" H 5150 3050 50  0001 C CNN
+F 2 "Capacitor_SMD:C_0805_2012Metric_Pad1.15x1.40mm_HandSolder" H 5150 3050 50  0001 C CNN
 F 3 "~" H 5150 3050 50  0001 C CNN
 	1    5150 3050
@@
 F 0 "R10" H 6068 3946 50  0000 L CNN
 F 1 "51K" H 6068 3855 50  0000 L CNN
-F 2 "" V 6040 3890 50  0001 C CNN
+F 2 "Resistor_SMD:R_0805_2012Metric_Pad1.15x1.40mm_HandSolder" V 6040 3890 50  0001 C CNN
 F 3 "~" H 6000 3900 50  0001 C CNN
 	1    6000 3900
@@
 F 0 "R9" H 6468 3746 50  0000 L CNN
 F 1 "470K" H 6468 3655 50  0000 L CNN
-F 2 "" V 6440 3690 50  0001 C CNN
+F 2 "Resistor_SMD:R_0805_2012Metric_Pad1.15x1.40mm_HandSolder" V 6440 3690 50  0001 C CNN
 F 3 "~" H 6400 3700 50  0001 C CNN
 	1    6400 3700
@@
 F 0 "R11" H 6468 4146 50  0000 L CNN
 F 1 "82K" H 6468 4055 50  0000 L CNN
-F 2 "" V 6440 4090 50  0001 C CNN
+F 2 "Resistor_SMD:R_0805_2012Metric_Pad1.15x1.40mm_HandSolder" V 6440 4090 50  0001 C CNN
 F 3 "~" H 6400 4100 50  0001 C CNN
 	1    6400 4100
@@
 	1    0    0    -1
 $EndComp
+$Comp
+L smi:LT1460 U1
+U 1 1 5DCD09A4
+P 3800 2600
+F 0 "U1" H 3800 2865 50  0000 C CNN
+F 1 "LT1460" H 3800 2774 50  0000 C CNN
+F 2 "TO_SOT_Packages_SMD:SOT-23_Handsoldering" H 3800 2600 50  0001 C CNN
+F 3 "" H 3800 2600 50  0001 C CNN
+	1    3800 2600
+	1    0    0    -1
+$EndComp
+$Comp
+L power:GNDPWR #PWR0117
+U 1 1 5DCD0B5E
+P 3800 3100
+F 0 "#PWR0117" H 3800 2900 50  0001 C CNN
+F 1 "GNDPWR" H 3804 2946 50  0000 C CNN
+F 2 "" H 3800 3050 50  0001 C CNN
+F 3 "" H 3800 3050 50  0001 C CNN
+	1    3800 3100
+	1    0    0    -1
+$EndComp
+Wire Wire Line
+	4250 2600 5450 2600
+Wire Wire Line
+	5450 2600 5450 3050
+Wire Wire Line
+	5450 2500 5450 2600
+Connection ~ 5450 2600
+$Comp
+L smi:+18V #U0101
+U 1 1 5DCD0E4C
+P 3050 2300
+F 0 "#U0101" H 3050 2300 50  0001 C CNN
+F 1 "+18V" H 3108 2287 50  0000 L CNN
+F 2 "" H 3050 2300 50  0001 C CNN
+F 3 "" H 3050 2300 50  0001 C CNN
+	1    3050 2300
+	1    0    0    -1
+$EndComp
+Wire Wire Line
+	3050 2350 3050 2600
+Wire Wire Line
+	3050 2600 3350 2600
 $EndSCHEMATC
