File: hardware/analog/smi_filter.sch (KiCad schematic (older format))
At the start: 25 parts, among them U11 TL082, U14 TL081, U15 TL082

Commit message: Nail down component values for filter
Parts:
- added JP?: DC disconnect, symbol Jumper:SolderJumper_2_Open
- C14: value C_Small -> 1uF
- C17, C18: value C_Small -> 47pF
- C21, C22: value C_Small -> 680pF
- R17: value R_US -> 8.2K
- R18, R20: value R_US -> 51K
- R19, R21: value R_US -> 9.1K
- R22: value 23K5 -> 23.5K
- R24, R26: value R_US -> 13K
- R25, R27: value R_US -> 180K
Connections:
- wire segments 86 -> 87
Other:
- note added: "4-pole Butterworth Filter (Sallen Key Biquadratic Pair)\nCutoff frequency: 41.3KHz\nDamping: 0.9969\nDC gain: 14.83 per stage\n"
- note added: "If we need to revert to our old setup, the\nsolder jumper can be disconnected and\na wire can be run from the TIA to the\noutput instead."
- note added: "Passive High Pass\n3dB point: 0.67 Hz"
- note added: "Passive Low Pass\n3dB point: 20Hz"
- note added: "Total gain: 22000"
- note removed: "4-pole Butterworth Filter (Sallen Key Biquadratic Pair)"
Changed lines of the file:
@@
 AR Path="/5D8F6AE1/5DA8AE19/5DA8BA7D" Ref="R22"  Part="1"
 F 0 "R22" H 3868 4796 50  0000 L CNN
-F 1 "23K5" H 3868 4705 50  0000 L CNN
+F 1 "23.5K" H 3868 4705 50  0000 L CNN
 F 2 "" V 3840 4740 50  0001 C CNN
 F 3 "~" H 3800 4750 50  0001 C CNN
@@
 P 4750 4400
 F 0 "R18" V 4545 4400 50  0000 C CNN
-F 1 "R_US" V 4636 4400 50  0000 C CNN
+F 1 "51K" V 4636 4400 50  0000 C CNN
 F 2 "" V 4790 4390 50  0001 C CNN
 F 3 "~" H 4750 4400 50  0001 C CNN
@@
 P 5200 4400
 F 0 "R19" V 4995 4400 50  0000 C CNN
-F 1 "R_US" V 5086 4400 50  0000 C CNN
+F 1 "9.1K" V 5086 4400 50  0000 C CNN
 F 2 "" V 5240 4390 50  0001 C CNN
 F 3 "~" H 5200 4400 50  0001 C CNN
@@
 P 5850 3800
 F 0 "C17" V 5621 3800 50  0000 C CNN
-F 1 "C_Small" V 5712 3800 50  0000 C CNN
+F 1 "47pF" V 5712 3800 50  0000 C CNN
 F 2 "" H 5850 3800 50  0001 C CNN
 F 3 "~" H 5850 3800 50  0001 C CNN
@@
 P 6300 5150
 F 0 "R25" V 6400 5150 50  0000 C CNN
-F 1 "R_US" V 6500 5150 50  0000 C CNN
+F 1 "180K" V 6500 5150 50  0000 C CNN
 F 2 "" V 6340 5140 50  0001 C CNN
 F 3 "~" H 6300 5150 50  0001 C CNN
@@
 P 5450 4600
 F 0 "C21" H 5542 4646 50  0000 L CNN
-F 1 "C_Small" H 5542 4555 50  0000 L CNN
+F 1 "680pF" H 5542 4555 50  0000 L CNN
 F 2 "" H 5450 4600 50  0001 C CNN
 F 3 "~" H 5450 4600 50  0001 C CNN
@@
 P 5500 5150
 F 0 "R24" V 5600 5150 50  0000 C CNN
-F 1 "R_US" V 5700 5150 50  0000 C CNN
+F 1 "13K" V 5700 5150 50  0000 C CNN
 F 2 "" V 5540 5140 50  0001 C CNN
 F 3 "~" H 5500 5150 50  0001 C CNN
@@
 P 7150 4500
 F 0 "R20" V 6945 4500 50  0000 C CNN
-F 1 "R_US" V 7036 4500 50  0000 C CNN
+F 1 "51K" V 7036 4500 50  0000 C CNN
 F 2 "" V 7190 4490 50  0001 C CNN
 F 3 "~" H 7150 4500 50  0001 C CNN
@@
 P 7650 4500
 F 0 "R21" V 7445 4500 50  0000 C CNN
-F 1 "R_US" V 7536 4500 50  0000 C CNN
+F 1 "9.1K" V 7536 4500 50  0000 C CNN
 F 2 "" V 7690 4490 50  0001 C CNN
 F 3 "~" H 7650 4500 50  0001 C CNN
@@
 P 7900 4700
 F 0 "C22" H 7992 4746 50  0000 L CNN
-F 1 "C_Small" H 7992 4655 50  0000 L CNN
+F 1 "680pF" H 7992 4655 50  0000 L CNN
 F 2 "" H 7900 4700 50  0001 C CNN
 F 3 "~" H 7900 4700 50  0001 C CNN
@@
 P 8950 5400
 F 0 "R27" V 8745 5400 50  0000 C CNN
-F 1 "R_US" V 8836 5400 50  0000 C CNN
+F 1 "180K" V 8836 5400 50  0000 C CNN
 F 2 "" V 8990 5390 50  0001 C CNN
 F 3 "~" H 8950 5400 50  0001 C CNN
@@
 P 8200 5400
 F 0 "R26" V 7995 5400 50  0000 C CNN
-F 1 "R_US" V 8086 5400 50  0000 C CNN
+F 1 "13K" V 8086 5400 50  0000 C CNN
 F 2 "" V 8240 5390 50  0001 C CNN
 F 3 "~" H 8200 5400 50  0001 C CNN
@@
 P 8750 3850
 F 0 "C18" V 8521 3850 50  0000 C CNN
-F 1 "C_Small" V 8612 3850 50  0000 C CNN
+F 1 "47pF" V 8612 3850 50  0000 C CNN
 F 2 "" H 8750 3850 50  0001 C CNN
 F 3 "~" H 8750 3850 50  0001 C CNN
@@
 P 6300 2100
 F 0 "C14" H 6392 2146 50  0000 L CNN
-F 1 "C_Small" H 6392 2055 50  0000 L CNN
+F 1 "1uF" H 6392 2055 50  0000 L CNN
 F 2 "" H 6300 2100 50  0001 C CNN
 F 3 "~" H 6300 2100 50  0001 C CNN
@@
 P 5800 1800
 F 0 "R17" V 5595 1800 50  0000 C CNN
-F 1 "R_US" V 5686 1800 50  0000 C CNN
+F 1 "8.2K" V 5686 1800 50  0000 C CNN
 F 2 "" V 5840 1790 50  0001 C CNN
 F 3 "~" H 5800 1800 50  0001 C CNN
@@
 Wire Wire Line
 	6750 1800 6300 1800
-Wire Wire Line
-	3600 1700 3600 4400
-Wire Wire Line
-	3450 4400 3600 4400
-Connection ~ 3600 4400
-Wire Wire Line
-	3600 4400 3800 4400
 $Comp
 L power:+9V #PWR027
@@
 Wire Wire Line
 	9400 2650 9250 2650
-Text Notes 4950 5800 0    50   ~ 0
-4-pole Butterworth Filter (Sallen Key Biquadratic Pair)
+Text Notes 4950 6050 0    50   ~ 0
+4-pole Butterworth Filter (Sallen Key Biquadratic Pair)\nCutoff frequency: 41.3KHz\nDamping: 0.9969\nDC gain: 14.83 per stage\n
 Wire Wire Line
 	5400 1800 5650 1800
@@
 Wire Wire Line
 	6300 1800 5950 1800
+$Comp
+L Jumper:SolderJumper_2_Open JP?
+U 1 1 5DBBC2A1
+P 3600 3200
+F 0 "JP?" V 3554 3268 50  0000 L CNN
+F 1 "DC disconnect" V 3645 3268 50  0000 L CNN
+F 2 "" H 3600 3200 50  0001 C CNN
+F 3 "~" H 3600 3200 50  0001 C CNN
+	1    3600 3200
+	0    1    1    0
+$EndComp
+Wire Wire Line
+	3600 1700 3600 3050
+Wire Wire Line
+	3600 3350 3600 4400
+Connection ~ 3600 4400
+Wire Wire Line
+	3600 4400 3800 4400
+Wire Wire Line
+	3450 4400 3600 4400
+Wire Notes Line
+	3650 4100 3650 5150
+Wire Notes Line
+	3650 5150 4400 5150
+Wire Notes Line
+	4400 5150 4400 4100
+Wire Notes Line
+	4400 4100 3650 4100
+Text Notes 3650 5350 0    50   ~ 0
+Passive High Pass\n3dB point: 0.67 Hz
+Text Notes 6000 1750 0    50   ~ 0
+Passive Low Pass\n3dB point: 20Hz
+Text Notes 3700 3650 0    50   ~ 0
+If we need to revert to our old setup, the\nsolder jumper can be disconnected and\na wire can be run from the TIA to the\noutput instead.
+Text Notes 9850 4050 0    50   ~ 0
+Total gain: 22000
 $EndSCHEMATC

Commit message: Save filters and whatnot before the culling
TODO:
- split ambient and SMI circuitry onto different boards
- kill off the pseudoground and use lipo batteries instead
Parts:
- removed JP?: DC disconnect, symbol Jumper:SolderJumper_2_Open
- C13, C14, C16, C17, C18, C19, C20, C21, C22: footprint (none) -> Capacitor_SMD:C_0805_2012Metric_Pad1.15x1.40mm_HandSolder
- C25, C26: renamed from C?; footprint (none) -> Capacitor_SMD:C_0805_2012Metric_Pad1.15x1.40mm_HandSolder
- R17, R18, R19, R20, R21, R23, R24, R25, R26, R27: footprint (none) -> Resistor_SMD:R_0805_2012Metric_Pad1.15x1.40mm_HandSolder
- R22: value 23.5K -> 22K; footprint (none) -> Resistor_SMD:R_0805_2012Metric_Pad1.15x1.40mm_HandSolder
- U11, U14: footprint (none) -> Housings_SOIC:SOIC-8_3.9x4.9mm_Pitch1.27mm
- U15: footprint (none) -> Housings_SOIC:SOIC-8-1EP_3.9x4.9mm_Pitch1.27mm
Connections:
- wire segments 87 -> 86
Other:
- note added: "Passive High Pass\n3dB point: 0.72 Hz"
- note removed: "If we need to revert to our old setup, the\nsolder jumper can be disconnected and\na wire can be run from the TIA to the\noutput instead."
- note removed: "Passive High Pass\n3dB point: 0.67 Hz"
- moved on the sheet: U11B, U15B
