File: hardware/analog/temperature.sch (KiCad schematic (older format))
At the start: 8 parts, among them U04 +18V, U05 +18V, U6 INA125P

Commit message: Refine analog circuitry
Parts:
- removed U04, U05: +18V, symbol smi:+18V
- added C?: 0.1uF, symbol Device:C_Small
Connections:
- net labels added: +9V, -9V, GNDREF
- net labels removed: GNDPWR
- wire segments 36 -> 41
Changed lines of the file:
@@
 $Descr A4 11693 8268
 encoding utf-8
-Sheet 3 6
+Sheet 5 7
 Title ""
 Date ""
@@
 AR Path="/5D8EE9F6/5D8F05C2" Ref="U6"  Part="1"
 AR Path="/5D8EEFE9/5D8F05C2" Ref="U10"  Part="1"
-F 0 "U6" H 6200 3100 50  0000 C CNN
+F 0 "U10" H 6200 3100 50  0000 C CNN
 F 1 "INA125P" H 6200 3000 50  0000 C CNN
 F 2 "" H 7650 1450 50  0001 C CNN
@@
 AR Path="/5D8EE9F6/5D8F06D7" Ref="R5"  Part="1"
 AR Path="/5D8EEFE9/5D8F06D7" Ref="R12"  Part="1"
-F 0 "R5" H 3668 3696 50  0000 L CNN
+F 0 "R12" H 3668 3696 50  0000 L CNN
 F 1 "330K" H 3668 3605 50  0000 L CNN
 F 2 "" V 3640 3640 50  0001 C CNN
@@
 AR Path="/5D8EE9F6/5D8F0741" Ref="R6"  Part="1"
 AR Path="/5D8EEFE9/5D8F0741" Ref="R13"  Part="1"
-F 0 "R6" H 4118 3696 50  0000 L CNN
+F 0 "R13" H 4118 3696 50  0000 L CNN
 F 1 "1K1" H 4118 3605 50  0000 L CNN
 F 2 "" V 4090 3640 50  0001 C CNN
@@
 AR Path="/5D8EE9F6/5D8F07C5" Ref="R8"  Part="1"
 AR Path="/5D8EEFE9/5D8F07C5" Ref="R15"  Part="1"
-F 0 "R8" H 3668 4296 50  0000 L CNN
+F 0 "R15" H 3668 4296 50  0000 L CNN
 F 1 "3K3" H 3668 4205 50  0000 L CNN
 F 2 "" V 3640 4240 50  0001 C CNN
@@
 Wire Wire Line
 	3850 4600 3600 4600
-$Comp
-L power:GNDPWR #PWR014
-U 1 1 5D8F3ED9
-P 3850 4750
-AR Path="/5D8EE9F6/5D8F3ED9" Ref="#PWR014"  Part="1"
-AR Path="/5D8EEFE9/5D8F3ED9" Ref="#PWR021"  Part="1"
-F 0 "#PWR014" H 3850 4550 50  0001 C CNN
-F 1 "GNDPWR" H 3854 4596 50  0000 C CNN
-F 2 "" H 3850 4700 50  0001 C CNN
-F 3 "" H 3850 4700 50  0001 C CNN
-	1    3850 4750
-	1    0    0    -1
-$EndComp
 Wire Wire Line
 	3600 3500 3600 3400
@@
 	3600 3900 3600 3800
 Connection ~ 3600 3900
-$Comp
-L power:GNDPWR #PWR013
-U 1 1 5D8F4488
-P 5950 4650
-AR Path="/5D8EE9F6/5D8F4488" Ref="#PWR013"  Part="1"
-AR Path="/5D8EEFE9/5D8F4488" Ref="#PWR020"  Part="1"
-F 0 "#PWR013" H 5950 4450 50  0001 C CNN
-F 1 "GNDPWR" H 5954 4496 50  0000 C CNN
-F 2 "" H 5950 4600 50  0001 C CNN
-F 3 "" H 5950 4600 50  0001 C CNN
-	1    5950 4650
-	1    0    0    -1
-$EndComp
-$Comp
-L smi:+18V U04
-U 1 1 5D8F4534
-P 5950 2400
-AR Path="/5D8EE9F6/5D8F4534" Ref="U04"  Part="1"
-AR Path="/5D8EEFE9/5D8F4534" Ref="U08"  Part="1"
-F 0 "U04" H 5950 2400 50  0001 C CNN
-F 1 "+18V" H 6008 2387 50  0000 L CNN
-F 2 "" H 5950 2400 50  0001 C CNN
-F 3 "" H 5950 2400 50  0001 C CNN
-	1    5950 2400
-	1    0    0    -1
-$EndComp
 Wire Wire Line
 	5950 2450 5950 2650
@@
 AR Path="/5D8EE9F6/5D8F47C5" Ref="C8"  Part="1"
 AR Path="/5D8EEFE9/5D8F47C5" Ref="C10"  Part="1"
-F 0 "C8" V 5371 2650 50  0000 C CNN
+F 0 "C10" V 5371 2650 50  0000 C CNN
 F 1 "0.1uF" V 5462 2650 50  0000 C CNN
 F 2 "" H 5600 2650 50  0001 C CNN
@@
 Wire Wire Line
 	5950 2650 5950 2750
-$Comp
-L power:GNDPWR #PWR012
-U 1 1 5D8F4A11
-P 6700 4450
-AR Path="/5D8EE9F6/5D8F4A11" Ref="#PWR012"  Part="1"
-AR Path="/5D8EEFE9/5D8F4A11" Ref="#PWR019"  Part="1"
-F 0 "#PWR012" H 6700 4250 50  0001 C CNN
-F 1 "GNDPWR" H 6704 4296 50  0000 C CNN
-F 2 "" H 6700 4400 50  0001 C CNN
-F 3 "" H 6700 4400 50  0001 C CNN
-	1    6700 4450
-	1    0    0    -1
-$EndComp
 Wire Wire Line
 	6700 4450 6700 4200
@@
 AR Path="/5D8EE9F6/5D8F4EAF" Ref="R7"  Part="1"
 AR Path="/5D8EEFE9/5D8F4EAF" Ref="R14"  Part="1"
-F 0 "R7" H 7218 3996 50  0000 L CNN
+F 0 "R14" H 7218 3996 50  0000 L CNN
 F 1 "2K" H 7218 3905 50  0000 L CNN
 F 2 "" V 7190 3940 50  0001 C CNN
@@
 Wire Wire Line
 	6750 3400 6550 3400
-$Comp
-L smi:+18V U05
-U 1 1 5D8F5B70
-P 6550 2750
-AR Path="/5D8EE9F6/5D8F5B70" Ref="U05"  Part="1"
-AR Path="/5D8EEFE9/5D8F5B70" Ref="U09"  Part="1"
-F 0 "U05" H 6550 2750 50  0001 C CNN
-F 1 "+18V" H 6608 2737 50  0000 L CNN
-F 2 "" H 6550 2750 50  0001 C CNN
-F 3 "" H 6550 2750 50  0001 C CNN
-	1    6550 2750
-	1    0    0    -1
-$EndComp
 Wire Wire Line
 	6550 2800 6550 3200
-$Comp
-L power:GNDPWR #PWR011
-U 1 1 5D8F613B
-P 5200 2750
-AR Path="/5D8EE9F6/5D8F613B" Ref="#PWR011"  Part="1"
-AR Path="/5D8EEFE9/5D8F613B" Ref="#PWR018"  Part="1"
-F 0 "#PWR011" H 5200 2550 50  0001 C CNN
-F 1 "GNDPWR" H 5204 2596 50  0000 C CNN
-F 2 "" H 5200 2700 50  0001 C CNN
-F 3 "" H 5200 2700 50  0001 C CNN
-	1    5200 2750
-	1    0    0    -1
-$EndComp
 Wire Wire Line
 	5200 2750 5200 2650
@@
 Text Notes 5600 5350 0    50   ~ 0
 TODO: fix grounding
+$Comp
+L power:GNDREF #PWR012
+U 1 1 5D9238FF
+P 6700 4450
+AR Path="/5D8EE9F6/5D9238FF" Ref="#PWR012"  Part="1"
+AR Path="/5D8EEFE9/5D9238FF" Ref="#PWR019"  Part="1"
+F 0 "#PWR019" H 6700 4200 50  0001 C CNN
+F 1 "GNDREF" H 6705 4277 50  0000 C CNN
+F 2 "" H 6700 4450 50  0001 C CNN
+F 3 "" H 6700 4450 50  0001 C CNN
+	1    6700 4450
+	1    0    0    -1
+$EndComp
+$Comp
+L power:+9V #PWR?
+U 1 1 5DBB1E67
+P 5950 2450
+AR Path="/5D8EE9F6/5DBB1E67" Ref="#PWR?"  Part="1"
+AR Path="/5D8EEFE9/5DBB1E67" Ref="#PWR?"  Part="1"
+F 0 "#PWR?" H 5950 2300 50  0001 C CNN
+F 1 "+9V" H 5965 2623 50  0000 C CNN
+F 2 "" H 5950 2450 50  0001 C CNN
+F 3 "" H 5950 2450 50  0001 C CNN
+	1    5950 2450
+	1    0    0    -1
+$EndComp
+$Comp
+L power:GNDREF #PWR?
+U 1 1 5DBB1FAF
+P 5200 2750
+AR Path="/5D8EE9F6/5DBB1FAF" Ref="#PWR?"  Part="1"
+AR Path="/5D8EEFE9/5DBB1FAF" Ref="#PWR?"  Part="1"
+F 0 "#PWR?" H 5200 2500 50  0001 C CNN
+F 1 "GNDREF" H 5205 2577 50  0000 C CNN
+F 2 "" H 5200 2750 50  0001 C CNN
+F 3 "" H 5200 2750 50  0001 C CNN
+	1    5200 2750
+	1    0    0    -1
+$EndComp
+$Comp
+L power:GNDREF #PWR?
+U 1 1 5DBB38AB
+P 3850 4750
+F 0 "#PWR?" H 3850 4500 50  0001 C CNN
+F 1 "GNDREF" H 3855 4577 50  0000 C CNN
+F 2 "" H 3850 4750 50  0001 C CNN
+F 3 "" H 3850 4750 50  0001 C CNN
+	1    3850 4750
+	1    0    0    -1
+$EndComp
+$Comp
+L power:-9V #PWR?
+U 1 1 5DBB39B6
+P 5950 5000
+F 0 "#PWR?" H 5950 4875 50  0001 C CNN
+F 1 "-9V" H 5965 5173 50  0000 C CNN
+F 2 "" H 5950 5000 50  0001 C CNN
+F 3 "" H 5950 5000 50  0001 C CNN
+	1    5950 5000
+	-1   0    0    1
+$EndComp
+$Comp
+L Device:C_Small C?
+U 1 1 5DBB3F53
+P 5600 4800
+AR Path="/5D8EE9F6/5DBB3F53" Ref="C?"  Part="1"
+AR Path="/5D8EEFE9/5DBB3F53" Ref="C?"  Part="1"
+F 0 "C?" V 5371 4800 50  0000 C CNN
+F 1 "0.1uF" V 5462 4800 50  0000 C CNN
+F 2 "" H 5600 4800 50  0001 C CNN
+F 3 "~" H 5600 4800 50  0001 C CNN
+	1    5600 4800
+	0    1    1    0
+$EndComp
+Wire Wire Line
+	5700 4800 5950 4800
+Wire Wire Line
+	5950 4650 5950 4800
+Connection ~ 5950 4800
+Wire Wire Line
+	5950 4800 5950 5000
+$Comp
+L power:GNDREF #PWR?
+U 1 1 5DBB4BBC
+P 5350 4950
+F 0 "#PWR?" H 5350 4700 50  0001 C CNN
+F 1 "GNDREF" H 5355 4777 50  0000 C CNN
+F 2 "" H 5350 4950 50  0001 C CNN
+F 3 "" H 5350 4950 50  0001 C CNN
+	1    5350 4950
+	1    0    0    -1
+$EndComp
+Wire Wire Line
+	5350 4950 5350 4800
+Wire Wire Line
+	5350 4800 5500 4800
+$Comp
+L power:+9V #PWR?
+U 1 1 5DBB54BC
+P 6550 2800
+F 0 "#PWR?" H 6550 2650 50  0001 C CNN
+F 1 "+9V" H 6565 2973 50  0000 C CNN
+F 2 "" H 6550 2800 50  0001 C CNN
+F 3 "" H 6550 2800 50  0001 C CNN
+	1    6550 2800
+	1    0    0    -1
+$EndComp
 $EndSCHEMATC

Commit message: Save filters and whatnot before the culling
TODO:
- split ambient and SMI circuitry onto different boards
- kill off the pseudoground and use lipo batteries instead
Parts:
- C23: renamed from C?; footprint (none) -> Capacitor_SMD:C_0805_2012Metric_Pad1.15x1.40mm_HandSolder
- C8: footprint (none) -> Capacitor_SMD:C_0805_2012Metric_Pad1.15x1.40mm_HandSolder
- R5, R6, R7, R8: footprint (none) -> Resistor_SMD:R_0805_2012Metric_Pad1.15x1.40mm_HandSolder
- U6: footprint (none) -> Housings_SOIC:SOIC-16_3.9x9.9mm_Pitch1.27mm
Changed lines of the file:
@@
 AR Path="/5D8EE9F6/5D8F05C2" Ref="U6"  Part="1"
 AR Path="/5D8EEFE9/5D8F05C2" Ref="U10"  Part="1"
-F 0 "U10" H 6200 3100 50  0000 C CNN
+F 0 "U6" H 6200 3100 50  0000 C CNN
 F 1 "INA125P" H 6200 3000 50  0000 C CNN
-F 2 "" H 7650 1450 50  0001 C CNN
+F 2 "Housings_SOIC:SOIC-16_3.9x9.9mm_Pitch1.27mm" H 7650 1450 50  0001 C CNN
 F 3 "" H 7650 1450 50  0001 C CNN
 	1    5950 2950
@@
 AR Path="/5D8EE9F6/5D8F06D7" Ref="R5"  Part="1"
 AR Path="/5D8EEFE9/5D8F06D7" Ref="R12"  Part="1"
-F 0 "R12" H 3668 3696 50  0000 L CNN
+F 0 "R5" H 3668 3696 50  0000 L CNN
 F 1 "330K" H 3668 3605 50  0000 L CNN
-F 2 "" V 3640 3640 50  0001 C CNN
+F 2 "Resistor_SMD:R_0805_2012Metric_Pad1.15x1.40mm_HandSolder" V 3640 3640 50  0001 C CNN
 F 3 "~" H 3600 3650 50  0001 C CNN
 	1    3600 3650
@@
 AR Path="/5D8EE9F6/5D8F0741" Ref="R6"  Part="1"
 AR Path="/5D8EEFE9/5D8F0741" Ref="R13"  Part="1"
-F 0 "R13" H 4118 3696 50  0000 L CNN
+F 0 "R6" H 4118 3696 50  0000 L CNN
 F 1 "1K1" H 4118 3605 50  0000 L CNN
-F 2 "" V 4090 3640 50  0001 C CNN
+F 2 "Resistor_SMD:R_0805_2012Metric_Pad1.15x1.40mm_HandSolder" V 4090 3640 50  0001 C CNN
 F 3 "~" H 4050 3650 50  0001 C CNN
 	1    4050 3650
@@
 AR Path="/5D8EE9F6/5D8F07C5" Ref="R8"  Part="1"
 AR Path="/5D8EEFE9/5D8F07C5" Ref="R15"  Part="1"
-F 0 "R15" H 3668 4296 50  0000 L CNN
+F 0 "R8" H 3668 4296 50  0000 L CNN
 F 1 "3K3" H 3668 4205 50  0000 L CNN
-F 2 "" V 3640 4240 50  0001 C CNN
+F 2 "Resistor_SMD:R_0805_2012Metric_Pad1.15x1.40mm_HandSolder" V 3640 4240 50  0001 C CNN
 F 3 "~" H 3600 4250 50  0001 C CNN
 	1    3600 4250
@@
 AR Path="/5D8EE9F6/5D8F47C5" Ref="C8"  Part="1"
 AR Path="/5D8EEFE9/5D8F47C5" Ref="C10"  Part="1"
-F 0 "C10" V 5371 2650 50  0000 C CNN
+F 0 "C8" V 5371 2650 50  0000 C CNN
 F 1 "0.1uF" V 5462 2650 50  0000 C CNN
-F 2 "" H 5600 2650 50  0001 C CNN
+F 2 "Capacitor_SMD:C_0805_2012Metric_Pad1.15x1.40mm_HandSolder" H 5600 2650 50  0001 C CNN
 F 3 "~" H 5600 2650 50  0001 C CNN
 	1    5600 2650
@@
 AR Path="/5D8EE9F6/5D8F4EAF" Ref="R7"  Part="1"
 AR Path="/5D8EEFE9/5D8F4EAF" Ref="R14"  Part="1"
-F 0 "R14" H 7218 3996 50  0000 L CNN
+F 0 "R7" H 7218 3996 50  0000 L CNN
 F 1 "2K" H 7218 3905 50  0000 L CNN
-F 2 "" V 7190 3940 50  0001 C CNN
+F 2 "Resistor_SMD:R_0805_2012Metric_Pad1.15x1.40mm_HandSolder" V 7190 3940 50  0001 C CNN
 F 3 "~" H 7150 3950 50  0001 C CNN
 	1    7150 3950
@@
 AR Path="/5D8EE9F6/5D9238FF" Ref="#PWR012"  Part="1"
 AR Path="/5D8EEFE9/5D9238FF" Ref="#PWR019"  Part="1"
-F 0 "#PWR019" H 6700 4200 50  0001 C CNN
+F 0 "#PWR012" H 6700 4200 50  0001 C CNN
 F 1 "GNDREF" H 6705 4277 50  0000 C CNN
 F 2 "" H 6700 4450 50  0001 C CNN
@@
 $EndComp
 $Comp
-L power:+9V #PWR?
+L power:+9V #PWR0101
 U 1 1 5DBB1E67
 P 5950 2450
-AR Path="/5D8EE9F6/5DBB1E67" Ref="#PWR?"  Part="1"
-AR Path="/5D8EEFE9/5DBB1E67" Ref="#PWR?"  Part="1"
-F 0 "#PWR?" H 5950 2300 50  0001 C CNN
+AR Path="/5D8EE9F6/5DBB1E67" Ref="#PWR0101"  Part="1"
+AR Path="/5D8EEFE9/5DBB1E67" Ref="#PWR0107"  Part="1"
+F 0 "#PWR0101" H 5950 2300 50  0001 C CNN
 F 1 "+9V" H 5965 2623 50  0000 C CNN
 F 2 "" H 5950 2450 50  0001 C CNN
@@
 $EndComp
 $Comp
-L power:GNDREF #PWR?
+L power:GNDREF #PWR0102
 U 1 1 5DBB1FAF
 P 5200 2750
-AR Path="/5D8EE9F6/5DBB1FAF" Ref="#PWR?"  Part="1"
-AR Path="/5D8EEFE9/5DBB1FAF" Ref="#PWR?"  Part="1"
-F 0 "#PWR?" H 5200 2500 50  0001 C CNN
+AR Path="/5D8EE9F6/5DBB1FAF" Ref="#PWR0102"  Part="1"
+AR Path="/5D8EEFE9/5DBB1FAF" Ref="#PWR0108"  Part="1"
+F 0 "#PWR0102" H 5200 2500 50  0001 C CNN
 F 1 "GNDREF" H 5205 2577 50  0000 C CNN
 F 2 "" H 5200 2750 50  0001 C CNN
@@
 $EndComp
 $Comp
-L power:GNDREF #PWR?
+L power:GNDREF #PWR0103
 U 1 1 5DBB38AB
 P 3850 4750
-F 0 "#PWR?" H 3850 4500 50  0001 C CNN
+AR Path="/5D8EE9F6/5DBB38AB" Ref="#PWR0103"  Part="1"
+AR Path="/5D8EEFE9/5DBB38AB" Ref="#PWR0109"  Part="1"
+F 0 "#PWR0103" H 3850 4500 50  0001 C CNN
 F 1 "GNDREF" H 3855 4577 50  0000 C CNN
 F 2 "" H 3850 4750 50  0001 C CNN
@@
 $EndComp
 $Comp
-L power:-9V #PWR?
+L power:-9V #PWR0104
 U 1 1 5DBB39B6
 P 5950 5000
-F 0 "#PWR?" H 5950 4875 50  0001 C CNN
+AR Path="/5D8EE9F6/5DBB39B6" Ref="#PWR0104"  Part="1"
+AR Path="/5D8EEFE9/5DBB39B6" Ref="#PWR0110"  Part="1"
+F 0 "#PWR0104" H 5950 4875 50  0001 C CNN
 F 1 "-9V" H 5965 5173 50  0000 C CNN
 F 2 "" H 5950 5000 50  0001 C CNN
@@
 $EndComp
 $Comp
-L Device:C_Small C?
+L Device:C_Small C23
 U 1 1 5DBB3F53
 P 5600 4800
-AR Path="/5D8EE9F6/5DBB3F53" Ref="C?"  Part="1"
-AR Path="/5D8EEFE9/5DBB3F53" Ref="C?"  Part="1"
-F 0 "C?" V 5371 4800 50  0000 C CNN
+AR Path="/5D8EE9F6/5DBB3F53" Ref="C23"  Part="1"
+AR Path="/5D8EEFE9/5DBB3F53" Ref="C24"  Part="1"
+F 0 "C23" V 5371 4800 50  0000 C CNN
 F 1 "0.1uF" V 5462 4800 50  0000 C CNN
-F 2 "" H 5600 4800 50  0001 C CNN
+F 2 "Capacitor_SMD:C_0805_2012Metric_Pad1.15x1.40mm_HandSolder" H 5600 4800 50  0001 C CNN
 F 3 "~" H 5600 4800 50  0001 C CNN
 	1    5600 4800
@@
 	5950 4800 5950 5000
 $Comp
-L power:GNDREF #PWR?
+L power:GNDREF #PWR0105
 U 1 1 5DBB4BBC
 P 5350 4950
-F 0 "#PWR?" H 5350 4700 50  0001 C CNN
+AR Path="/5D8EE9F6/5DBB4BBC" Ref="#PWR0105"  Part="1"
+AR Path="/5D8EEFE9/5DBB4BBC" Ref="#PWR0111"  Part="1"
+F 0 "#PWR0105" H 5350 4700 50  0001 C CNN
 F 1 "GNDREF" H 5355 4777 50  0000 C CNN
 F 2 "" H 5350 4950 50  0001 C CNN
@@
 	5350 4800 5500 4800
 $Comp
-L power:+9V #PWR?
+L power:+9V #PWR0106
 U 1 1 5DBB54BC
 P 6550 2800
-F 0 "#PWR?" H 6550 2650 50  0001 C CNN
+AR Path="/5D8EE9F6/5DBB54BC" Ref="#PWR0106"  Part="1"
+AR Path="/5D8EEFE9/5DBB54BC" Ref="#PWR0112"  Part="1"
+F 0 "#PWR0106" H 6550 2650 50  0001 C CNN
 F 1 "+9V" H 6565 2973 50  0000 C CNN
 F 2 "" H 6550 2800 50  0001 C CNN
