File: hardware/prototype/prototype.kicad_pcb (KiCad board)
At the start: 2 copper layers, 47 x 52.7 mm, 16 parts, among them J1 OUTPUT probe, J2 BATT HIGH, J3 OUTPUT, J4 BATT LOW, J5 LASER CONN, U1 TL082, U2 LT1460-5

Commit message: Update prototype PCB
Parts:
- added G***: LOGO, hardware:logo_25mm, F.Cu at (115.1, 59.2)
- added H1: MountingHole, Mounting_Holes:MountingHole_3.2mm_M3_Pad, F.Cu at (71.1, 42.5)
- added H2: MountingHole, Mounting_Holes:MountingHole_3.2mm_M3_Pad, F.Cu at (71.1, 87.0)
- added H3: MountingHole, Mounting_Holes:MountingHole_3.2mm_M3_Pad, F.Cu at (115.6, 42.5)
- added H4: MountingHole, Mounting_Holes:MountingHole_3.2mm_M3_Pad, F.Cu at (115.6, 87.0)
- moved J5 2.54 mm to (80.0, 45.7)
- moved J3 2.54 mm to (94.0, 45.7)
- moved J2 1.54 mm to (94.6, 83.8)
- moved J4 1.50 mm to (105.7, 83.8)
Routing:
- net /TIA_OUT: track 56.7 -> 58.8 mm
- net /LD_IN: track 38.9 -> 40.2 mm
Other:
- board size 47 x 52.7 mm -> 53.3 x 53.3 mm
