File: hardware/smi_board/smi_filter.sch (KiCad schematic (older format))
At the start: 25 parts, among them U11 TL082, U14 TL081, U15 TL082

Commit message: Split monolithic board into ambient and smi
Connections:
- net labels added: +12V, -12V, GND
- net labels removed: +9V, -9V, GNDREF
