File: hardware/ambient/ambient.sch (KiCad schematic (older format))
At the start: 14 parts, among them J1 BATT+, J2 DAQ CONN, J3 BATT-, J4 RTD CONN, J5 RTD CONN, J6 RTD CONN, J7 RTD CONN, U1 AZ1117-5.0

Commit message: Add layout for ambient sensors
Parts:
- C1, C12: footprint (none) -> Capacitor_THT:CP_Radial_D5.0mm_P2.50mm
- H1, H2, H3, H4: footprint (none) -> MountingHole:MountingHole_3.2mm_M3_Pad
- J1, J3: footprint (none) -> Connector_Phoenix_MC:PhoenixContact_MCV_1,5_2-G-3.5_1x02_P3.50mm_Vertical
- J2: footprint (none) -> Connector_Phoenix_MC:PhoenixContact_MCV_1,5_7-G-3.5_1x07_P3.50mm_Vertical
- J4, J5, J6, J7: footprint (none) -> Connector_JST:JST_EH_S02B-EH_1x02_P2.50mm_Horizontal
- U1: footprint (none) -> Package_TO_SOT_SMD:SOT-223-3_TabPin2
Changed lines of the file:
@@
 F 0 "J1" H 1494 1485 50  0000 C CNN
 F 1 "BATT+" H 1494 1394 50  0000 C CNN
-F 2 "" H 1600 1300 50  0001 C CNN
+F 2 "Connector_Phoenix_MC:PhoenixContact_MCV_1,5_2-G-3.5_1x02_P3.50mm_Vertical" H 1600 1300 50  0001 C CNN
 F 3 "~" H 1600 1300 50  0001 C CNN
 	1    1600 1300
@@
 F 0 "J3" H 1494 1985 50  0000 C CNN
 F 1 "BATT-" H 1494 1894 50  0000 C CNN
-F 2 "" H 1600 1800 50  0001 C CNN
+F 2 "Connector_Phoenix_MC:PhoenixContact_MCV_1,5_2-G-3.5_1x02_P3.50mm_Vertical" H 1600 1800 50  0001 C CNN
 F 3 "~" H 1600 1800 50  0001 C CNN
 	1    1600 1800
@@
 F 0 "J7" H 6078 6176 50  0000 L CNN
 F 1 "RTD CONN" H 6078 6085 50  0000 L CNN
-F 2 "" H 6050 6200 50  0001 C CNN
+F 2 "Connector_JST:JST_EH_S02B-EH_1x02_P2.50mm_Horizontal" H 6050 6200 50  0001 C CNN
 F 3 "~" H 6050 6200 50  0001 C CNN
 	1    6050 6200
@@
 F 0 "J6" H 6078 4726 50  0000 L CNN
 F 1 "RTD CONN" H 6078 4635 50  0000 L CNN
-F 2 "" H 6050 4750 50  0001 C CNN
+F 2 "Connector_JST:JST_EH_S02B-EH_1x02_P2.50mm_Horizontal" H 6050 4750 50  0001 C CNN
 F 3 "~" H 6050 4750 50  0001 C CNN
 	1    6050 4750
@@
 F 0 "J5" H 6078 3276 50  0000 L CNN
 F 1 "RTD CONN" H 6078 3185 50  0000 L CNN
-F 2 "" H 6050 3300 50  0001 C CNN
+F 2 "Connector_JST:JST_EH_S02B-EH_1x02_P2.50mm_Horizontal" H 6050 3300 50  0001 C CNN
 F 3 "~" H 6050 3300 50  0001 C CNN
 	1    6050 3300
@@
 F 0 "J4" H 6078 1826 50  0000 L CNN
 F 1 "RTD CONN" H 6078 1735 50  0000 L CNN
-F 2 "" H 6050 1850 50  0001 C CNN
+F 2 "Connector_JST:JST_EH_S02B-EH_1x02_P2.50mm_Horizontal" H 6050 1850 50  0001 C CNN
 F 3 "~" H 6050 1850 50  0001 C CNN
 	1    6050 1850
@@
 	6050 4350 5850 4350
 Text Label 6000 5800 0    50   ~ 0
-RTD_AMP_3
+RTD_AMP_4
 Wire Wire Line
 	6000 5800 5850 5800
@@
 F 0 "J2" H 9177 1726 50  0000 L CNN
 F 1 "DAQ CONN" H 9177 1635 50  0000 L CNN
-F 2 "" H 9150 1700 50  0001 C CNN
+F 2 "Connector_Phoenix_MC:PhoenixContact_MCV_1,5_7-G-3.5_1x07_P3.50mm_Vertical" H 9150 1700 50  0001 C CNN
 F 3 "~" H 9150 1700 50  0001 C CNN
 	1    9150 1700
@@
 Wire Wire Line
 	8900 2000 8950 2000
+Text Label 8650 1600 2    50   ~ 0
+RTD_AMP_1
+Text Label 8650 1700 2    50   ~ 0
+RTD_AMP_2
+Text Label 8650 1800 2    50   ~ 0
+RTD_AMP_3
+Text Label 8650 1900 2    50   ~ 0
+RTD_AMP_4
 Text Label 8650 1400 2    50   ~ 0
-RTD_AMP_1
+PRESSURE
 Text Label 8650 1500 2    50   ~ 0
-RTD_AMP_2
-Text Label 8650 1600 2    50   ~ 0
-RTD_AMP_3
-Text Label 8650 1700 2    50   ~ 0
-RTD_AMP_4
-Text Label 8650 1800 2    50   ~ 0
-PRESSURE
-Text Label 8650 1900 2    50   ~ 0
 PRESSURE_BK
 Wire Wire Line
@@
 F 0 "U1" H 2250 3392 50  0000 C CNN
 F 1 "AZ1117-5.0" H 2250 3301 50  0000 C CNN
-F 2 "" H 2250 3400 50  0001 C CIN
+F 2 "Package_TO_SOT_SMD:SOT-223-3_TabPin2" H 2250 3400 50  0001 C CIN
 F 3 "https://www.diodes.com/assets/Datasheets/AZ1117.pdf" H 2250 3150 50  0001 C CNN
 	1    2250 3150
@@
 F 0 "C1" H 1615 3346 50  0000 L CNN
 F 1 "10uF" H 1615 3255 50  0000 L CNN
-F 2 "" H 1538 3150 50  0001 C CNN
+F 2 "Capacitor_THT:CP_Radial_D5.0mm_P2.50mm" H 1538 3150 50  0001 C CNN
 F 3 "~" H 1500 3300 50  0001 C CNN
 	1    1500 3300
@@
 F 0 "C12" H 3065 3346 50  0000 L CNN
 F 1 "22uF" H 3065 3255 50  0000 L CNN
-F 2 "" H 2988 3150 50  0001 C CNN
+F 2 "Capacitor_THT:CP_Radial_D5.0mm_P2.50mm" H 2988 3150 50  0001 C CNN
 F 3 "~" H 2950 3300 50  0001 C CNN
 	1    2950 3300
@@
 F 0 "H1" H 8150 5446 50  0000 L CNN
 F 1 "MountingHole" H 8150 5355 50  0000 L CNN
-F 2 "" H 8050 5400 50  0001 C CNN
+F 2 "MountingHole:MountingHole_3.2mm_M3_Pad" H 8050 5400 50  0001 C CNN
 F 3 "~" H 8050 5400 50  0001 C CNN
 	1    8050 5400
@@
 F 0 "H3" H 8150 5796 50  0000 L CNN
 F 1 "MountingHole" H 8150 5705 50  0000 L CNN
-F 2 "" H 8050 5750 50  0001 C CNN
+F 2 "MountingHole:MountingHole_3.2mm_M3_Pad" H 8050 5750 50  0001 C CNN
 F 3 "~" H 8050 5750 50  0001 C CNN
 	1    8050 5750
@@
 F 0 "H2" H 9000 5446 50  0000 L CNN
 F 1 "MountingHole" H 9000 5355 50  0000 L CNN
-F 2 "" H 8900 5400 50  0001 C CNN
+F 2 "MountingHole:MountingHole_3.2mm_M3_Pad" H 8900 5400 50  0001 C CNN
 F 3 "~" H 8900 5400 50  0001 C CNN
 	1    8900 5400
@@
 F 0 "H4" H 9000 5796 50  0000 L CNN
 F 1 "MountingHole" H 9000 5705 50  0000 L CNN
-F 2 "" H 8900 5750 50  0001 C CNN
+F 2 "MountingHole:MountingHole_3.2mm_M3_Pad" H 8900 5750 50  0001 C CNN
 F 3 "~" H 8900 5750 50  0001 C CNN
 	1    8900 5750
