File: hardware/ambient/pressure.sch (KiCad schematic (older format))
At the start: 9 parts, among them U6 MPXA6115A, U7 TL082, U8 MPXA6115A

Commit message: Add layout for ambient sensors
Parts:
- added C13, C14: 0.1uF, Capacitor_SMD:C_0805_2012Metric_Pad1.15x1.40mm_HandSolder, symbol Device:C
- added unit 3 of U7
- C10, C11: value C_Small -> 0.1uF
- U7: footprint (none) -> Housings_SOIC:SOIC-8_3.9x4.9mm_Pitch1.27mm
Connections:
- net labels added: +12V, -12V, P_BK_RAW, P_RAW
- wire segments 36 -> 42
Changed lines of the file:
@@
 AR Path="/5DD1C8AB/5D8EF91F" Ref="C10"  Part="1"
 F 0 "C10" V 3671 1900 50  0000 C CNN
-F 1 "C_Small" V 3762 1900 50  0000 C CNN
+F 1 "0.1uF" V 3762 1900 50  0000 C CNN
 F 2 "Capacitor_SMD:C_0805_2012Metric_Pad1.15x1.40mm_HandSolder" H 3900 1900 50  0001 C CNN
 F 3 "~" H 3900 1900 50  0001 C CNN
@@
 AR Path="/5DD1C8AB/5DD1F681" Ref="C11"  Part="1"
 F 0 "C11" V 3621 4550 50  0000 C CNN
-F 1 "C_Small" V 3712 4550 50  0000 C CNN
+F 1 "0.1uF" V 3712 4550 50  0000 C CNN
 F 2 "Capacitor_SMD:C_0805_2012Metric_Pad1.15x1.40mm_HandSolder" H 3850 4550 50  0001 C CNN
 F 3 "~" H 3850 4550 50  0001 C CNN
@@
 F 0 "U7" H 6000 3217 50  0000 C CNN
 F 1 "TL082" H 6000 3126 50  0000 C CNN
-F 2 "" H 6000 2850 50  0001 C CNN
+F 2 "Housings_SOIC:SOIC-8_3.9x4.9mm_Pitch1.27mm" H 6000 2850 50  0001 C CNN
 F 3 "http://www.ti.com/lit/ds/symlink/tl081.pdf" H 6000 2850 50  0001 C CNN
 	1    6000 2850
@@
 F 0 "U7" H 5950 5867 50  0000 C CNN
 F 1 "TL082" H 5950 5776 50  0000 C CNN
-F 2 "" H 5950 5500 50  0001 C CNN
+F 2 "Housings_SOIC:SOIC-8_3.9x4.9mm_Pitch1.27mm" H 5950 5500 50  0001 C CNN
 F 3 "http://www.ti.com/lit/ds/symlink/tl081.pdf" H 5950 5500 50  0001 C CNN
 	2    5950 5500
@@
 Text Notes 7550 2950 0    50   ~ 0
 Buffer the output of the sensor\nto prevent crosstalk on the DAQ
+$Comp
+L Amplifier_Operational:TL082 U7
+U 3 1 5DD2EEE4
+P 8450 4300
+F 0 "U7" H 8408 4346 50  0000 L CNN
+F 1 "TL082" H 8408 4255 50  0000 L CNN
+F 2 "Housings_SOIC:SOIC-8_3.9x4.9mm_Pitch1.27mm" H 8450 4300 50  0001 C CNN
+F 3 "http://www.ti.com/lit/ds/symlink/tl081.pdf" H 8450 4300 50  0001 C CNN
+	3    8450 4300
+	1    0    0    -1
+$EndComp
+$Comp
+L power:+12V #PWR0101
+U 1 1 5DD2EF8E
+P 8350 3800
+F 0 "#PWR0101" H 8350 3650 50  0001 C CNN
+F 1 "+12V" H 8365 3973 50  0000 C CNN
+F 2 "" H 8350 3800 50  0001 C CNN
+F 3 "" H 8350 3800 50  0001 C CNN
+	1    8350 3800
+	1    0    0    -1
+$EndComp
+Wire Wire Line
+	8350 3800 8350 3900
+$Comp
+L power:-12V #PWR0102
+U 1 1 5DD2F545
+P 8350 4800
+F 0 "#PWR0102" H 8350 4900 50  0001 C CNN
+F 1 "-12V" H 8365 4973 50  0000 C CNN
+F 2 "" H 8350 4800 50  0001 C CNN
+F 3 "" H 8350 4800 50  0001 C CNN
+	1    8350 4800
+	-1   0    0    1
+$EndComp
+Wire Wire Line
+	8350 4800 8350 4700
+$Comp
+L Device:C C13
+U 1 1 5DD2FB2C
+P 8950 3900
+F 0 "C13" V 8698 3900 50  0000 C CNN
+F 1 "0.1uF" V 8789 3900 50  0000 C CNN
+F 2 "Capacitor_SMD:C_0805_2012Metric_Pad1.15x1.40mm_HandSolder" H 8988 3750 50  0001 C CNN
+F 3 "~" H 8950 3900 50  0001 C CNN
+	1    8950 3900
+	0    1    1    0
+$EndComp
+$Comp
+L power:GND #PWR0103
+U 1 1 5DD2FC89
+P 9100 3900
+F 0 "#PWR0103" H 9100 3650 50  0001 C CNN
+F 1 "GND" H 9105 3727 50  0000 C CNN
+F 2 "" H 9100 3900 50  0001 C CNN
+F 3 "" H 9100 3900 50  0001 C CNN
+	1    9100 3900
+	1    0    0    -1
+$EndComp
+Wire Wire Line
+	8800 3900 8350 3900
+Connection ~ 8350 3900
+Wire Wire Line
+	8350 3900 8350 4000
+$Comp
+L Device:C C14
+U 1 1 5DD3026B
+P 8950 4700
+F 0 "C14" V 8698 4700 50  0000 C CNN
+F 1 "0.1uF" V 8789 4700 50  0000 C CNN
+F 2 "Capacitor_SMD:C_0805_2012Metric_Pad1.15x1.40mm_HandSolder" H 8988 4550 50  0001 C CNN
+F 3 "~" H 8950 4700 50  0001 C CNN
+	1    8950 4700
+	0    1    1    0
+$EndComp
+$Comp
+L power:GND #PWR0104
+U 1 1 5DD30272
+P 9100 4700
+F 0 "#PWR0104" H 9100 4450 50  0001 C CNN
+F 1 "GND" H 9105 4527 50  0000 C CNN
+F 2 "" H 9100 4700 50  0001 C CNN
+F 3 "" H 9100 4700 50  0001 C CNN
+	1    9100 4700
+	1    0    0    -1
+$EndComp
+Wire Wire Line
+	8800 4700 8350 4700
+Connection ~ 8350 4700
+Wire Wire Line
+	8350 4700 8350 4600
+Text Label 5250 5400 0    50   ~ 0
+P_BK_RAW
+Text Label 5350 2750 0    50   ~ 0
+P_RAW
 $EndSCHEMATC
